File: Hardware/mainboard_bare_minimum_design/HM_mainboard/Microcontroller.kicad_sch (KiCad schematic)
At the start: 22 parts, among them J6 USB_C_Receptacle, Q2 MBT3904DW1T1, U1 ESP32-WROOM-E, U4 FT231XS, Y1 32.768 kHz

Commit message: Updated Comment
Other:
- note added: "Microcontroller and Bluetooth Module"
- note removed: "Microcontroller"
Changed lines of the file:
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@@
     (effects (font (size 2.54 2.159) (thickness 0.4318) bold) (justify left bottom))
   )
-  (text "Microcontroller\n" (at 19.05 119.38 0)
+  (text "Microcontroller and Bluetooth Module\n" (at 19.05 119.38 0)
     (effects (font (size 2.54 2.159) (thickness 0.4318) bold) (justify left bottom))
   )
