File: Hardware/mainboard_bare_minimum_design/HM_mainboard/untitled.kicad_sch (KiCad schematic)
At the start: 15 parts, among them Q1 MOSFET-PCHANNELDMG2307L, U2 V_REG_LDOSMD, U3 MCP73831

Commit message: Updated Comment
Changed lines of the file:
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@@
     (effects (font (size 2.032 1.7272)) (justify right bottom))
   )
-  (text "Lithium-Polymer Battery Charger (1-cell)" (at 58.42 116.84 0)
-    (effects (font (size 2.54 2.159)) (justify left top))
+  (text "Lithium-Polymer Battery Charger (1-cell)" (at 24.13 116.84 0)
+    (effects (font (size 2.54 2.54) (thickness 0.508) bold) (justify left bottom))
   )
   (text "Power Switch \n(see page UI-peripherals)" (at 73.66 66.04 0)
@@
     (effects (font (size 1.778 1.5113)) (justify top))
   )
-  (text "Voltage Regulator" (at 71.12 24.13 0)
-    (effects (font (size 2.54 2.159)) (justify left bottom))
+  (text "Voltage Regulator" (at 24.13 25.4 0)
+    (effects (font (size 2.54 2.54) (thickness 0.508) bold) (justify left bottom))
   )
   (text "SJ1 can be cut to\nmodify the charge-\ncurrent programming\nresistor."
