File: Hardware/HM_mainboard/UI_Peripherals.kicad_sch (KiCad schematic)
At the start: 16 parts, among them J3 54-00174, J4 54-00174, J5 54-00174, J6 54-00174, U4 WE-TVS-824015043

Commit message: Started component placement for PCB
Parts:
- U4: footprint Package_TO_SOT_SMD:SOT-23-6 -> Package_TO_SOT_SMD:SOT-23-6_Handsoldering
- renumbered D4 to D3, D5 to D4, J3 to J5, J5 to J6, J6 to J7
Changed lines of the file:
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@@
         )
         (path "/54a6df43-5475-46a2-9916-8b0260700d4c/137c5701-d01e-40ce-919d-b371cfda41da"
-          (reference "#PWR036") (unit 1)
+          (reference "#PWR032") (unit 1)
         )
       )
@@
         )
         (path "/54a6df43-5475-46a2-9916-8b0260700d4c/137c5701-d01e-40ce-919d-b371cfda41da"
-          (reference "#PWR033") (unit 1)
+          (reference "#PWR020") (unit 1)
         )
       )
@@
   (symbol (lib_id "Device:LED_Dual_KAK") (at 120.65 137.16 270) (unit 1)
     (in_bom yes) (on_board yes) (dnp no) (fields_autoplaced)
-    (property "Reference" "D5" (at 128.27 135.9535 90)
+    (property "Reference" "D4" (at 128.27 135.9535 90)
       (effects (font (size 1.27 1.27)) (justify left))
     )
@@
       (project "HM_mainboard"
         (path "/54a6df43-5475-46a2-9916-8b0260700d4c/137c5701-d01e-40ce-919d-b371cfda41da"
-          (reference "D5") (unit 1)
+          (reference "D4") (unit 1)
         )
       )
@@
         )
         (path "/54a6df43-5475-46a2-9916-8b0260700d4c/137c5701-d01e-40ce-919d-b371cfda41da"
-          (reference "#PWR023") (unit 1)
+          (reference "#PWR029") (unit 1)
         )
       )
@@
       (effects (font (size 1.27 1.27)) (justify left))
     )
-    (property "Footprint" "Package_TO_SOT_SMD:SOT-23-6" (at 247.65 146.05 0)
+    (property "Footprint" "Package_TO_SOT_SMD:SOT-23-6_Handsoldering" (at 247.65 146.05 0)
       (effects (font (size 1.27 1.27)) hide)
     )
@@
         )
         (path "/54a6df43-5475-46a2-9916-8b0260700d4c/137c5701-d01e-40ce-919d-b371cfda41da"
-          (reference "#PWR017") (unit 1)
+          (reference "#PWR021") (unit 1)
         )
       )
@@
         )
         (path "/54a6df43-5475-46a2-9916-8b0260700d4c/137c5701-d01e-40ce-919d-b371cfda41da"
-          (reference "#PWR019") (unit 1)
+          (reference "#PWR023") (unit 1)
         )
       )
@@
         )
         (path "/54a6df43-5475-46a2-9916-8b0260700d4c/137c5701-d01e-40ce-919d-b371cfda41da"
-          (reference "R11") (unit 1)
+          (reference "R10") (unit 1)
         )
       )
@@
         )
         (path "/54a6df43-5475-46a2-9916-8b0260700d4c/137c5701-d01e-40ce-919d-b371cfda41da"
-          (reference "#PWR034") (unit 1)
+          (reference "#PWR027") (unit 1)
         )
       )
@@
   (symbol (lib_id "HeadMouse:54-00174") (at 233.68 50.8 0) (unit 1)
     (in_bom yes) (on_board yes) (dnp no) (fields_autoplaced)
-    (property "Reference" "J6" (at 219.71 45.72 0)
+    (property "Reference" "J7" (at 219.71 45.72 0)
       (effects (font (size 1.524 1.524)))
     )
@@
       (project "HM_mainboard"
         (path "/54a6df43-5475-46a2-9916-8b0260700d4c/137c5701-d01e-40ce-919d-b371cfda41da"
-          (reference "J6") (unit 1)
+          (reference "J7") (unit 1)
         )
       )
@@
         )
         (path "/54a6df43-5475-46a2-9916-8b0260700d4c/137c5701-d01e-40ce-919d-b371cfda41da"
-          (reference "R10") (unit 1)
+          (reference "R9") (unit 1)
         )
       )
@@
         )
         (path "/54a6df43-5475-46a2-9916-8b0260700d4c/137c5701-d01e-40ce-919d-b371cfda41da"
-          (reference "#PWR020") (unit 1)
+          (reference "#PWR025") (unit 1)
         )
       )
@@
         )
         (path "/54a6df43-5475-46a2-9916-8b0260700d4c/137c5701-d01e-40ce-919d-b371cfda41da"
-          (reference "#PWR018") (unit 1)
+          (reference "#PWR022") (unit 1)
         )
       )
@@
         )
         (path "/54a6df43-5475-46a2-9916-8b0260700d4c/137c5701-d01e-40ce-919d-b371cfda41da"
-          (reference "#PWR024") (unit 1)
+          (reference "#PWR030") (unit 1)
         )
       )
@@
         )
         (path "/54a6df43-5475-46a2-9916-8b0260700d4c/137c5701-d01e-40ce-919d-b371cfda41da"
-          (reference "#PWR026") (unit 1)
+          (reference "#PWR033") (unit 1)
         )
       )
@@
         )
         (path "/54a6df43-5475-46a2-9916-8b0260700d4c/137c5701-d01e-40ce-919d-b371cfda41da"
-          (reference "C8") (unit 1)
+          (reference "C12") (unit 1)
         )
       )
@@
   (symbol (lib_id "HeadMouse:54-00174") (at 172.72 50.8 0) (unit 1)
     (in_bom yes) (on_board yes) (dnp no) (fields_autoplaced)
-    (property "Reference" "J5" (at 158.75 45.72 0)
+    (property "Reference" "J6" (at 158.75 45.72 0)
       (effects (font (size 1.524 1.524)))
     )
@@
       (project "HM_mainboard"
         (path "/54a6df43-5475-46a2-9916-8b0260700d4c/137c5701-d01e-40ce-919d-b371cfda41da"
-          (reference "J5") (unit 1)
+          (reference "J6") (unit 1)
         )
       )
@@
         )
         (path "/54a6df43-5475-46a2-9916-8b0260700d4c/137c5701-d01e-40ce-919d-b371cfda41da"
-          (reference "#SUPPLY013") (unit 1)
+          (reference "#SUPPLY014") (unit 1)
         )
       )
@@
         )
         (path "/54a6df43-5475-46a2-9916-8b0260700d4c/137c5701-d01e-40ce-919d-b371cfda41da"
-          (reference "C10") (unit 1)
+          (reference "C14") (unit 1)
         )
       )
@@
   (symbol (lib_id "HeadMouse:54-00174") (at 113.03 52.07 0) (unit 1)
     (in_bom yes) (on_board yes) (dnp no)
-    (property "Reference" "J3" (at 99.06 46.99 0)
+    (property "Reference" "J5" (at 99.06 46.99 0)
       (effects (font (size 1.524 1.524)))
     )
@@
       (project "HM_mainboard"
         (path "/54a6df43-5475-46a2-9916-8b0260700d4c/137c5701-d01e-40ce-919d-b371cfda41da"
-          (reference "J3") (unit 1)
+          (reference "J5") (unit 1)
         )
       )
@@
         )
         (path "/54a6df43-5475-46a2-9916-8b0260700d4c/137c5701-d01e-40ce-919d-b371cfda41da"
-          (reference "#PWR022") (unit 1)
+          (reference "#PWR028") (unit 1)
         )
       )
@@
         )
         (path "/54a6df43-5475-46a2-9916-8b0260700d4c/137c5701-d01e-40ce-919d-b371cfda41da"
-          (reference "#SUPPLY014") (unit 1)
+          (reference "#SUPPLY015") (unit 1)
         )
       )
@@
         )
         (path "/54a6df43-5475-46a2-9916-8b0260700d4c/137c5701-d01e-40ce-919d-b371cfda41da"
-          (reference "R9") (unit 1)
+          (reference "R8") (unit 1)
         )
       )
@@
         )
         (path "/54a6df43-5475-46a2-9916-8b0260700d4c/137c5701-d01e-40ce-919d-b371cfda41da"
-          (reference "#PWR025") (unit 1)
+          (reference "#PWR026") (unit 1)
         )
       )
@@
         )
         (path "/54a6df43-5475-46a2-9916-8b0260700d4c/137c5701-d01e-40ce-919d-b371cfda41da"
-          (reference "#PWR021") (unit 1)
+          (reference "#PWR024") (unit 1)
         )
       )
@@
         )
         (path "/54a6df43-5475-46a2-9916-8b0260700d4c/137c5701-d01e-40ce-919d-b371cfda41da"
-          (reference "#SUPPLY015") (unit 1)
+          (reference "#SUPPLY016") (unit 1)
         )
       )
@@
         )
         (path "/54a6df43-5475-46a2-9916-8b0260700d4c/137c5701-d01e-40ce-919d-b371cfda41da"
-          (reference "R12") (unit 1)
+          (reference "R11") (unit 1)
         )
       )
@@
         )
         (path "/54a6df43-5475-46a2-9916-8b0260700d4c/137c5701-d01e-40ce-919d-b371cfda41da"
-          (reference "C7") (unit 1)
+          (reference "C11") (unit 1)
         )
       )
@@
         )
         (path "/54a6df43-5475-46a2-9916-8b0260700d4c/137c5701-d01e-40ce-919d-b371cfda41da"
-          (reference "#PWR027") (unit 1)
+          (reference "#PWR034") (unit 1)
         )
       )
@@
         )
         (path "/54a6df43-5475-46a2-9916-8b0260700d4c/137c5701-d01e-40ce-919d-b371cfda41da"
-          (reference "C9") (unit 1)
+          (reference "C13") (unit 1)
         )
       )
@@
   (symbol (lib_id "Device:LED_Dual_KAK") (at 57.15 137.16 270) (unit 1)
     (in_bom yes) (on_board yes) (dnp no) (fields_autoplaced)
-    (property "Reference" "D4" (at 64.77 135.9535 90)
+    (property "Reference" "D3" (at 64.77 135.9535 90)
       (effects (font (size 1.27 1.27)) (justify left))
     )
@@
       (project "HM_mainboard"
         (path "/54a6df43-5475-46a2-9916-8b0260700d4c/137c5701-d01e-40ce-919d-b371cfda41da"
-          (reference "D4") (unit 1)
+          (reference "D3") (unit 1)
         )
       )
@@
         )
         (path "/54a6df43-5475-46a2-9916-8b0260700d4c/137c5701-d01e-40ce-919d-b371cfda41da"
-          (reference "#PWR035") (unit 1)
-        )
-      )
+          (reference "#PWR031") (unit 1)
+        )
+      )

Commit message: Updated footprint of auxiliary jacks, routed first version of PCB
Parts:
- J4, J5, J6, J7: footprint 54-00174_TEN -> HeadMouse:54-00174
Connections:
- net BTN_1: now also U4.3 (I/O2); no longer U4.1 (I/O1)
- net BTN_2: now also U4.1 (I/O1); no longer U4.3 (I/O2)
- net BTN_3: now also U4.6 (I/O4); no longer U4.4 (I/O3)
- net BTN_4: now also U4.4 (I/O3); no longer U4.6 (I/O4)
Changed lines of the file:
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@@
     (effects (font (size 1.27 1.27)) (justify left bottom))
   )
-  (label "TVS_BTN_3" (at 259.08 134.62 0) (fields_autoplaced)
+  (label "TVS_BTN_4" (at 259.08 134.62 0) (fields_autoplaced)
     (effects (font (size 1.27 1.27)) (justify left bottom))
   )
-  (label "TVS_BTN_2" (at 233.68 139.7 180) (fields_autoplaced)
+  (label "TVS_BTN_1" (at 233.68 139.7 180) (fields_autoplaced)
     (effects (font (size 1.27 1.27)) (justify right bottom))
   )
@@
     (effects (font (size 1.27 1.27)) (justify left bottom))
   )
-  (label "TVS_BTN_4" (at 259.08 139.7 0) (fields_autoplaced)
+  (label "TVS_BTN_3" (at 259.08 139.7 0) (fields_autoplaced)
     (effects (font (size 1.27 1.27)) (justify left bottom))
   )
-  (label "TVS_BTN_1" (at 233.68 134.62 180) (fields_autoplaced)
+  (label "TVS_BTN_2" (at 233.68 134.62 180) (fields_autoplaced)
     (effects (font (size 1.27 1.27)) (justify right bottom))
   )
@@
       (effects (font (size 1.524 1.524)))
     )
-    (property "Footprint" "54-00174_TEN" (at 233.68 50.8 0)
+    (property "Footprint" "HeadMouse:54-00174" (at 233.68 50.8 0)
       (effects (font (size 1.27 1.27) italic) hide)
     )
@@
       (effects (font (size 1.524 1.524)))
     )
-    (property "Footprint" "54-00174_TEN" (at 172.72 50.8 0)
+    (property "Footprint" "HeadMouse:54-00174" (at 172.72 50.8 0)
       (effects (font (size 1.27 1.27) italic) hide)
     )
@@
       (effects (font (size 1.524 1.524)))
     )
-    (property "Footprint" "54-00174_TEN" (at 113.03 52.07 0)
+    (property "Footprint" "HeadMouse:54-00174" (at 113.03 52.07 0)
       (effects (font (size 1.27 1.27) italic) hide)
     )
@@
       (effects (font (size 1.524 1.524)))
     )
-    (property "Footprint" "54-00174_TEN" (at 52.07 52.07 0)
+    (property "Footprint" "HeadMouse:54-00174" (at 52.07 52.07 0)
       (effects (font (size 1.27 1.27) italic) hide)
     )

Commit message: Added BOM
Parts:
- C6: value 100n -> 100nF
- D3, D4: Mouser (none) -> 155124RV73200; Mouser Price/Stock (none) -> https://www.mouser.at/ProductDetail/Wurth-Elektronik/155124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
- J4, J5, J6, J7: Digikey (none) -> 54-00174; Mouser Price/Stock (none) -> https://www.digikey.de/de/products/detail/tensility-interna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
- S3: Mouser (none) -> 450404015514
- U4: Mouser (none) -> 824015043; Mouser Price/Stock (none) -> https://www.mouser.at/ProductDetail/Wurth-Elektronik/824015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
Changed lines of the file:
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@@
+      (effects (font (size 1.27 1.27)) hide)
+    )
+    (property "Mouser" "155124RV73200" (at 120.65 137.16 0)
+      (effects (font (size 1.27 1.27)) hide)
+    )
+    (property "Mouser Price/Stock" "https://www.mouser.at/ProductDetail/Wurth-Elektronik/155124RV73200?qs=5aG0NVq1C4yQQzqaqWGYAg%3D%3D" (at 120.65 137.16 0)
+      (effects (font (size 1.27 1.27)) hide)
+    )
+    (property "Reichelt" "" (at 120.65 137.16 0)
       (effects (font (size 1.27 1.27)) hide)
     )
@@
       (effects (font (size 1.27 1.27)) hide)
     )
+    (property "Mouser" "824015043" (at 246.38 137.16 0)
+      (effects (font (size 1.27 1.27)) hide)
+    )
+    (property "Mouser Price/Stock" "https://www.mouser.at/ProductDetail/Wurth-Elektronik/824015043?qs=amGC7iS6iy%252BoHLfbVvujhQ%3D%3D" (at 246.38 137.16 0)
+      (effects (font (size 1.27 1.27)) hide)
+    )
+    (property "Reichelt" "" (at 246.38 137.16 0)
+      (effects (font (size 1.27 1.27)) hide)
+    )
     (pin "1")
     (pin "2")
@@
       (effects (font (size 1.27 1.27)) hide)
     )
+    (property "Reichelt" "" (at 118.11 153.67 0)
+      (effects (font (size 1.27 1.27)) hide)
+    )
     (pin "1")
     (pin "2")
@@
     (property "Manufacturer_Part_Number" "450404015514" (at 200.66 925.73 0)
       (effects (font (size 1.27 1.27)) (justify left top) hide)
+    )
+    (property "Mouser" "450404015514" (at 179.07 130.81 0)
+      (effects (font (size 1.27 1.27)) hide)
+    )
+    (property "Reichelt" "" (at 179.07 130.81 0)
+      (effects (font (size 1.27 1.27)) hide)
     )
     (pin "1")
@@
       (effects (font (size 1.27 1.27) italic) hide)
     )
-    (property "Datasheet" "54-00174" (at 233.68 50.8 0)
+    (property "Datasheet" "https://tensility.s3.amazonaws.com/uploads/pdffiles/54-00174.pdf?X-Amz-Expires=600&X-Amz-Date=20231206T211710Z&X-Amz-Algorithm=AWS4-HMAC-SHA256&X-Amz-Credential=AKIAIS2S4WRDQDSWDRZQ%2F20231206%2Fus-west-2%2Fs3%2Faws4_request&X-Amz-SignedHeaders=host&X-Amz-Signature=9b1a304331de7a209094883b10ea93c55c7e790e0be1d3e399b91f09e8b0233f" (at 233.68 50.8 0)
       (effects (font (size 1.27 1.27) italic) hide)
+    )
+    (property "Digikey" "54-00174" (at 233.68 50.8 0)
+      (effects (font (size 1.27 1.27)) hide)
+    )
+    (property "Mouser Price/Stock" "https://www.digikey.de/de/products/detail/tensility-international-corp/54-00174/12140150" (at 233.68 50.8 0)
+      (effects (font (size 1.27 1.27)) hide)
+    )
+    (property "Reichelt" "" (at 233.68 50.8 0)
+      (effects (font (size 1.27 1.27)) hide)
     )
     (pin "1")
@@
       (effects (font (size 1.27 1.27)) hide)
     )
+    (property "Reichelt" "" (at 59.69 152.4 0)
+      (effects (font (size 1.27 1.27)) hide)
+    )
     (pin "1")
     (pin "2")
@@
       (effects (font (size 1.27 1.27)) (justify left))
     )
-    (property "Value" "100n" (at 126.111 63.373 0)
+    (property "Value" "100nF" (at 126.111 63.373 0)
       (effects (font (size 1.27 1.27)) (justify left))
     )
@@
     )
     (property "RS Components" "200-6519" (at 123.19 62.23 0)
+      (effects (font (size 1.27 1.27)) hide)
+    )
+    (property "Reichelt" "" (at 123.19 62.23 0)
       (effects (font (size 1.27 1.27)) hide)
     )
@@
       (effects (font (size 1.27 1.27) italic) hide)
     )
-    (property "Datasheet" "54-00174" (at 172.72 50.8 0)
+    (property "Datasheet" "https://tensility.s3.amazonaws.com/uploads/pdffiles/54-00174.pdf?X-Amz-Expires=600&X-Amz-Date=20231206T211710Z&X-Amz-Algorithm=AWS4-HMAC-SHA256&X-Amz-Credential=AKIAIS2S4WRDQDSWDRZQ%2F20231206%2Fus-west-2%2Fs3%2Faws4_request&X-Amz-SignedHeaders=host&X-Amz-Signature=9b1a304331de7a209094883b10ea93c55c7e790e0be1d3e399b91f09e8b0233f" (at 172.72 50.8 0)
       (effects (font (size 1.27 1.27) italic) hide)
+    )
+    (property "Digikey" "54-00174" (at 172.72 50.8 0)
+      (effects (font (size 1.27 1.27)) hide)
+    )
+    (property "Mouser Price/Stock" "https://www.digikey.de/de/products/detail/tensility-international-corp/54-00174/12140150" (at 172.72 50.8 0)
+      (effects (font (size 1.27 1.27)) hide)
+    )
+    (property "Reichelt" "" (at 172.72 50.8 0)
+      (effects (font (size 1.27 1.27)) hide)
     )
     (pin "1")
@@
       (effects (font (size 1.27 1.27)) (justify left))
     )
-    (property "Value" "100n" (at 246.761 62.103 0)
+    (property "Value" "100nF" (at 246.761 62.103 0)
       (effects (font (size 1.27 1.27)) (justify left))
     )
@@
     )
     (property "RS Components" "200-6519" (at 243.84 60.96 0)
+      (effects (font (size 1.27 1.27)) hide)
+    )
+    (property "Reichelt" "" (at 243.84 60.96 0)
       (effects (font (size 1.27 1.27)) hide)
     )
@@
       (effects (font (size 1.27 1.27) italic) hide)
     )
-    (property "Datasheet" "54-00174" (at 113.03 52.07 0)
+    (property "Datasheet" "https://tensility.s3.amazonaws.com/uploads/pdffiles/54-00174.pdf?X-Amz-Expires=600&X-Amz-Date=20231206T211710Z&X-Amz-Algorithm=AWS4-HMAC-SHA256&X-Amz-Credential=AKIAIS2S4WRDQDSWDRZQ%2F20231206%2Fus-west-2%2Fs3%2Faws4_request&X-Amz-SignedHeaders=host&X-Amz-Signature=9b1a304331de7a209094883b10ea93c55c7e790e0be1d3e399b91f09e8b0233f" (at 113.03 52.07 0)
       (effects (font (size 1.27 1.27) italic) hide)
+    )
+    (property "Digikey" "54-00174" (at 113.03 52.07 0)
+      (effects (font (size 1.27 1.27)) hide)
+    )
+    (property "Mouser Price/Stock" "https://www.digikey.de/de/products/detail/tensility-international-corp/54-00174/12140150" (at 113.03 52.07 0)
+      (effects (font (size 1.27 1.27)) hide)
+    )
+    (property "Reichelt" "" (at 113.03 52.07 0)
+      (effects (font (size 1.27 1.27)) hide)
     )
     (pin "1")
@@
       (effects (font (size 1.27 1.27)) hide)
     )
+    (property "Reichelt" "" (at 54.61 152.4 0)
+      (effects (font (size 1.27 1.27)) hide)
+    )
     (pin "1")
     (pin "2")
@@
       (effects (font (size 1.27 1.27)) hide)
     )
+    (property "Reichelt" "" (at 123.19 153.67 0)
+      (effects (font (size 1.27 1.27)) hide)
+    )
     (pin "1")
     (pin "2")
@@
       (effects (font (size 1.27 1.27)) (justify left))
     )
-    (property "Value" "100n" (at 65.151 63.373 0)
+    (property "Value" "100nF" (at 65.151 63.373 0)
       (effects (font (size 1.27 1.27)) (justify left))
     )
@@
     )
     (property "RS Components" "200-6519" (at 62.23 62.23 0)
+      (effects (font (size 1.27 1.27)) hide)
+    )
+    (property "Reichelt" "" (at 62.23 62.23 0)
       (effects (font (size 1.27 1.27)) hide)
     )
@@
       (effects (font (size 1.27 1.27)) (justify left))
     )
-    (property "Value" "100n" (at 185.801 62.103 0)
+    (property "Value" "100nF" (at 185.801 62.103 0)
       (effects (font (size 1.27 1.27)) (justify left))
     )
@@
     )
     (property "RS Components" "200-6519" (at 182.88 60.96 0)
+      (effects (font (size 1.27 1.27)) hide)
+    )
+    (property "Reichelt" "" (at 182.88 60.96 0)
       (effects (font (size 1.27 1.27)) hide)
     )
@@
       (effects (font (size 1.27 1.27)) hide)
     )
+    (property "Mouser" "155124RV73200" (at 57.15 137.16 0)
+      (effects (font (size 1.27 1.27)) hide)
+    )
+    (property "Mouser Price/Stock" "https://www.mouser.at/ProductDetail/Wurth-Elektronik/155124RV73200?qs=5aG0NVq1C4yQQzqaqWGYAg%3D%3D" (at 57.15 137.16 0)
+      (effects (font (size 1.27 1.27)) hide)
+    )
+    (property "Reichelt" "" (at 57.15 137.16 0)
+      (effects (font (size 1.27 1.27)) hide)
+    )
     (pin "1")
     (pin "2")
@@
       (effects (font (size 1.27 1.27) italic) hide)
     )
-    (property "Datasheet" "54-00174" (at 52.07 52.07 0)
+    (property "Datasheet" "https://tensility.s3.amazonaws.com/uploads/pdffiles/54-00174.pdf?X-Amz-Expires=600&X-Amz-Date=20231206T211710Z&X-Amz-Algorithm=AWS4-HMAC-SHA256&X-Amz-Credential=AKIAIS2S4WRDQDSWDRZQ%2F20231206%2Fus-west-2%2Fs3%2Faws4_request&X-Amz-SignedHeaders=host&X-Amz-Signature=9b1a304331de7a209094883b10ea93c55c7e790e0be1d3e399b91f09e8b0233f" (at 52.07 52.07 0)
       (effects (font (size 1.27 1.27) italic) hide)
     )
-    (pin "1")
+    (property "Digikey" "54-00174" (at 52.07 52.07 0)
+      (effects (font (size 1.27 1.27)) hide)
+    )
+    (property "Mouser Price/Stock" "https://www.digikey.de/de/products/detail/tensility-international-corp/54-00174/12140150" (at 52.07 52.07 0)
+      (effects (font (size 1.27 1.27)) hide)
+    )
+    (property "Reichelt" "" (at 52.07 52.07 0)
+      (effects (font (size 1.27 1.27)) hide)
+    )
+    (pin "1")
