File: Hardware/HM_mainboard/UI_Peripherals.kicad_sch (KiCad schematic)
At the start: 16 parts, among them J4 54-00174, J5 54-00174, J6 54-00174, J7 54-00174, U4 WE-TVS-824015043

Commit message: Updated BOM
Parts:
- C6: Digikey 1276-CL10B104KB8NNNLCT-ND -> 1276-CL10B104KB8NNNLCT
- D3, D4: Mouser 155124RV73200 -> 710-155124RV73200
- J4, J5, J6, J7: Digikey 54-00174 -> 839-54-00174CT
- R6: Mouser ERJ-PA3J121V -> 603-RC0603FR-10120RL
- S3: Mouser 450404015514 -> 710-450404015514
- U4: Mouser 824015043 -> 710-824015043
Changed lines of the file:
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@@
       (effects (font (size 1.27 1.27)) hide)
     )
-    (property "Mouser" "155124RV73200" (at 120.65 137.16 0)
+    (property "Mouser" "710-155124RV73200" (at 120.65 137.16 0)
       (effects (font (size 1.27 1.27)) hide)
     )
@@
       (effects (font (size 1.27 1.27)) hide)
     )
-    (property "Mouser" "824015043" (at 246.38 137.16 0)
+    (property "Mouser" "710-824015043" (at 246.38 137.16 0)
       (effects (font (size 1.27 1.27)) hide)
     )
@@
       (effects (font (size 1.27 1.27)) hide)
     )
-    (property "Mouser" "ERJ-PA3J121V" (at 118.11 153.67 0)
+    (property "Mouser" "603-RC0603FR-10120RL" (at 118.11 153.67 0)
       (effects (font (size 1.27 1.27)) hide)
     )
@@
       (effects (font (size 1.27 1.27)) (justify left top) hide)
     )
-    (property "Mouser" "450404015514" (at 179.07 130.81 0)
+    (property "Mouser" "710-450404015514" (at 179.07 130.81 0)
       (effects (font (size 1.27 1.27)) hide)
     )
@@
       (effects (font (size 1.27 1.27) italic) hide)
     )
-    (property "Digikey" "54-00174" (at 233.68 50.8 0)
+    (property "Digikey" "839-54-00174CT" (at 233.68 50.8 0)
       (effects (font (size 1.27 1.27)) hide)
     )
@@
       (effects (font (size 1.27 1.27)) hide)
     )
-    (property "Mouser" "ERJ-PA3J121V" (at 59.69 152.4 0)
+    (property "Mouser" "603-RC0603FR-10120RL" (at 59.69 152.4 0)
       (effects (font (size 1.27 1.27)) hide)
     )
@@
       (effects (font (size 1.27 1.27)) hide)
     )
-    (property "Digikey" "1276-CL10B104KB8NNNLCT-ND" (at 123.19 62.23 0)
+    (property "Digikey" "1276-CL10B104KB8NNNLCT" (at 123.19 62.23 0)
       (effects (font (size 1.27 1.27)) hide)
     )
@@
       (effects (font (size 1.27 1.27) italic) hide)
     )
-    (property "Digikey" "54-00174" (at 172.72 50.8 0)
+    (property "Digikey" "839-54-00174CT" (at 172.72 50.8 0)
       (effects (font (size 1.27 1.27)) hide)
     )
@@
       (effects (font (size 1.27 1.27)) hide)
     )
-    (property "Digikey" "1276-CL10B104KB8NNNLCT-ND" (at 243.84 60.96 0)
+    (property "Digikey" "1276-CL10B104KB8NNNLCT" (at 243.84 60.96 0)
       (effects (font (size 1.27 1.27)) hide)
     )
@@
       (effects (font (size 1.27 1.27) italic) hide)
     )
-    (property "Digikey" "54-00174" (at 113.03 52.07 0)
+    (property "Digikey" "839-54-00174CT" (at 113.03 52.07 0)
       (effects (font (size 1.27 1.27)) hide)
     )
@@
       (effects (font (size 1.27 1.27)) hide)
     )
-    (property "Mouser" "ERJ-PA3J121V" (at 54.61 152.4 0)
+    (property "Mouser" "603-RC0603FR-10120RL" (at 54.61 152.4 0)
       (effects (font (size 1.27 1.27)) hide)
     )
@@
       (effects (font (size 1.27 1.27)) hide)
     )
-    (property "Mouser" "ERJ-PA3J121V" (at 123.19 153.67 0)
+    (property "Mouser" "603-RC0603FR-10120RL" (at 123.19 153.67 0)
       (effects (font (size 1.27 1.27)) hide)
     )
@@
       (effects (font (size 1.27 1.27)) hide)
     )
-    (property "Digikey" "1276-CL10B104KB8NNNLCT-ND" (at 62.23 62.23 0)
+    (property "Digikey" "1276-CL10B104KB8NNNLCT" (at 62.23 62.23 0)
       (effects (font (size 1.27 1.27)) hide)
     )
@@
       (effects (font (size 1.27 1.27)) hide)
     )
-    (property "Digikey" "1276-CL10B104KB8NNNLCT-ND" (at 182.88 60.96 0)
+    (property "Digikey" "1276-CL10B104KB8NNNLCT" (at 182.88 60.96 0)
       (effects (font (size 1.27 1.27)) hide)
     )
@@
       (effects (font (size 1.27 1.27)) hide)
     )
-    (property "Mouser" "155124RV73200" (at 57.15 137.16 0)
+    (property "Mouser" "710-155124RV73200" (at 57.15 137.16 0)
       (effects (font (size 1.27 1.27)) hide)
     )
@@
       (effects (font (size 1.27 1.27) italic) hide)
     )
-    (property "Digikey" "54-00174" (at 52.07 52.07 0)
-      (effects (font (size 1.27 1.27)) hide)
-    )
+    (property "Digikey" "839-54-00174CT" (at 52.07 52.07 0)
+      (effects (font (size 1.27 1.27)) hide)
+    )
