File: Hardware/HM_mainboard/Microcontroller.kicad_sch (KiCad schematic)
At the start: 17 parts, among them J2 USB4105-GF-A, J3 Conn_01x04, U3 ESP32-S3-WROOM-1, Y1 32.768 kHz

Commit message: Added BOM
Parts:
- C5: Digikey (none) -> 1276-CL10B104KB8NNNLCT-ND; Mouser (none) -> 581-06035C104K4; RS Components (none) -> 200-6519
- C5: value 1uF -> 1.0uF-25V-(+80/-20%); Mouser (none) -> F921E105KPA
- D2: Mouser (none) -> 824015; Mouser Price/Stock (none) -> https://www.mouser.at/ProductDetail/Wurth-Elektronik/824015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
- FL1: Mouser (none) -> 744232090; Mouser Price/Stock (none) -> https://www.mouser.at/ProductDetail/Wurth-Elektronik/744232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
- J2: Mouser (none) -> USB4105-GF-A; Mouser Price/Stock (none) -> https://www.mouser.at/ProductDetail/GCT/USB4105-GF-A?qs=KUo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
- J3: Mouser (none) -> Beliebige Stiftleiste, Raster: 2.54mm
- R10: Mouser (none) -> RN73H1JTTD5101F100; Mouser Price/Stock (none) -> https://www.mouser.at/ProductDetail/KOA-Speer/RN73H1JTTD510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
- S1, S2: Mouser (none) -> 13019315; Mouser Price/Stock (none) -> https://www.mouser.at/ProductDetail/Schurter/1301.9315?qs=t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
- U3: Mouser (none) -> ESP32-S3-WROOM-1-N8; Mouser Price/Stock (none) -> https://www.mouser.at/ProductDetail/Espressif-Systems/ESP32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
- Y1: Mouser (none) -> ASDK-32.768KHz-LRT; Mouser Price/Stock (none) -> https://www.mouser.at/ProductDetail/ABRACON/ABS07-32768KHZ-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
Changed lines of the file:
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@@
+      (effects (font (size 1.27 1.27)) hide)
+    )
+    (property "Reichelt" "" (at 121.92 95.25 0)
+      (effects (font (size 1.27 1.27)) hide)
+    )
+    (property "Digikey" "1276-CL10B104KB8NNNLCT-ND" (at 121.92 95.25 0)
+      (effects (font (size 1.27 1.27)) hide)
+    )
+    (property "Mouser" "581-06035C104K4" (at 121.92 95.25 0)
+      (effects (font (size 1.27 1.27)) hide)
+    )
+    (property "RS Components" "200-6519" (at 121.92 95.25 0)
       (effects (font (size 1.27 1.27)) hide)
     )
@@
     )
     (property "Datasheet" "~" (at 238.76 119.38 0)
+      (effects (font (size 1.27 1.27)) hide)
+    )
+    (property "Reichelt" "" (at 238.76 119.38 0)
+      (effects (font (size 1.27 1.27)) hide)
+    )
+    (property "Digikey" "1276-CL10B104KB8NNNLCT-ND" (at 238.76 119.38 0)
+      (effects (font (size 1.27 1.27)) hide)
+    )
+    (property "Mouser" "581-06035C104K4" (at 238.76 119.38 0)
+      (effects (font (size 1.27 1.27)) hide)
+    )
+    (property "RS Components" "200-6519" (at 238.76 119.38 0)
       (effects (font (size 1.27 1.27)) hide)
     )
@@
     )
     (property "Datasheet" "https://www.usb.org/sites/default/files/documents/usb_type-c.zip" (at 46.99 49.53 0)
+      (effects (font (size 1.27 1.27)) hide)
+    )
+    (property "Mouser" "USB4105-GF-A" (at 43.18 49.53 0)
+      (effects (font (size 1.27 1.27)) hide)
+    )
+    (property "Mouser Price/Stock" "https://www.mouser.at/ProductDetail/GCT/USB4105-GF-A?qs=KUoIvG%2F9IlY%2FMLlBMpStpA%3D%3D&gad_source=1&gclid=Cj0KCQiAyKurBhD5ARIsALamXaHB1WqEL8FpCW_cEPz8SMNbaXEcthQ5WIWoRdPENYKDcg-3_OVy5qsaArQwEALw_wcB" (at 43.18 49.53 0)
+      (effects (font (size 1.27 1.27)) hide)
+    )
+    (property "Reichelt" "" (at 43.18 49.53 0)
       (effects (font (size 1.27 1.27)) hide)
     )
@@
       (effects (font (size 1.27 1.27)) hide)
     )
+    (property "Reichelt" "" (at 67.31 39.37 0)
+      (effects (font (size 1.27 1.27)) hide)
+    )
+    (property "Mouser" "RN73H1JTTD5101F100" (at 67.31 39.37 0)
+      (effects (font (size 1.27 1.27)) hide)
+    )
+    (property "Mouser Price/Stock" "https://www.mouser.at/ProductDetail/KOA-Speer/RN73H1JTTD5101F100?qs=Tw8F%252BABiY2owhjU7td4KeQ%3D%3D" (at 67.31 39.37 0)
+      (effects (font (size 1.27 1.27)) hide)
+    )
     (pin "1")
     (pin "2")
@@
     )
     (property "Datasheet" "https://www.we-online.com/components/products/datasheet/824015.pdf" (at 161.29 53.34 0)
+      (effects (font (size 1.27 1.27)) hide)
+    )
+    (property "Mouser" "824015" (at 110.49 50.8 0)
+      (effects (font (size 1.27 1.27)) hide)
+    )
+    (property "Mouser Price/Stock" "https://www.mouser.at/ProductDetail/Wurth-Elektronik/824015?qs=Wn16VcyqZWp2%252Bq7OHpgqcg%3D%3D" (at 110.49 50.8 0)
+      (effects (font (size 1.27 1.27)) hide)
+    )
+    (property "Reichelt" "" (at 110.49 50.8 0)
       (effects (font (size 1.27 1.27)) hide)
     )
@@
       (effects (font (size 1.27 1.27)) hide)
     )
+    (property "Reichelt" "" (at 114.3 95.25 0)
+      (effects (font (size 1.27 1.27)) hide)
+    )
     (pin "1")
     (pin "2")
@@
     )
     (property "Datasheet" "https://www.espressif.com/sites/default/files/documentation/esp32-s3-wroom-1_wroom-1u_datasheet_en.pdf" (at 107.95 195.58 0)
+      (effects (font (size 1.27 1.27)) hide)
+    )
+    (property "Mouser" "ESP32-S3-WROOM-1-N8" (at 105.41 144.78 0)
+      (effects (font (size 1.27 1.27)) hide)
+    )
+    (property "Mouser Price/Stock" "https://www.mouser.at/ProductDetail/Espressif-Systems/ESP32-S3-WROOM-1-N8?qs=sGAEpiMZZMu3sxpa5v1qrpuLb1YRQvRH486xd1meH8w%3D" (at 105.41 144.78 0)
+      (effects (font (size 1.27 1.27)) hide)
+    )
+    (property "Reichelt" "" (at 105.41 144.78 0)
       (effects (font (size 1.27 1.27)) hide)
     )
@@
       (effects (font (size 1.27 1.27)) hide)
     )
+    (property "Reichelt" "" (at 250.19 106.68 0)
+      (effects (font (size 1.27 1.27)) hide)
+    )
     (pin "1")
     (pin "2")
@@
       (effects (font (size 1.27 1.27)) hide)
     )
+    (property "Mouser" "744232090" (at 151.13 50.8 0)
+      (effects (font (size 1.27 1.27)) hide)
+    )
+    (property "Mouser Price/Stock" "https://www.mouser.at/ProductDetail/Wurth-Elektronik/744232090?qs=PGXP4M47uW6L5fAiLO6yTw%3D%3D" (at 151.13 50.8 0)
+      (effects (font (size 1.27 1.27)) hide)
+    )
+    (property "Reichelt" "" (at 151.13 50.8 0)
+      (effects (font (size 1.27 1.27)) hide)
+    )
     (pin "1")
     (pin "2")
@@
       (effects (font (size 1.27 1.27)) hide)
     )
+    (property "Reichelt" "" (at 35.56 120.65 0)
+      (effects (font (size 1.27 1.27)) hide)
+    )
     (pin "1")
     (pin "2")
@@
       (effects (font (size 1.27 1.27)) (justify right))
     )
-    (property "Value" "1uF" (at 254 119.38 0)
+    (property "Value" "1.0uF-25V-(+80/-20%)" (at 254 119.38 0)
       (effects (font (size 1.27 1.27)) (justify right))
     )
@@
     )
     (property "Datasheet" "~" (at 250.19 118.11 0)
+      (effects (font (size 1.27 1.27)) hide)
+    )
+    (property "Mouser" "F921E105KPA" (at 250.19 118.11 0)
+      (effects (font (size 1.27 1.27)) hide)
+    )
+    (property "Reichelt" "" (at 250.19 118.11 0)
       (effects (font (size 1.27 1.27)) hide)
     )
@@
       (effects (font (size 1.27 1.27)) hide)
     )
+    (property "Mouser" "ASDK-32.768KHz-LRT" (at 40.64 118.11 0)
+      (effects (font (size 1.27 1.27)) hide)
+    )
+    (property "Mouser Price/Stock" "https://www.mouser.at/ProductDetail/ABRACON/ABS07-32768KHZ-T?qs=3SpAxaLJ01g8GJWeO3sA3Q%3D%3D&mgh=1&gad_source=1&gclid=CjwKCAiA9ourBhAVEiwA3L5RFmcTURdfJp_IENxutYTSDuJVwm7JT5lA7J1Dl65ASlIgL4B9Xx2CFxoCmaUQAvD_BwE" (at 40.64 118.11 0)
+      (effects (font (size 1.27 1.27)) hide)
+    )
+    (property "Reichelt" "" (at 40.64 118.11 0)
+      (effects (font (size 1.27 1.27)) hide)
+    )
     (pin "1")
     (pin "2")
@@
       (effects (font (size 1.27 1.27)) hide)
     )
+    (property "Reichelt" "" (at 203.2 66.675 0)
+      (effects (font (size 1.27 1.27)) hide)
+    )
+    (property "Mouser" "Beliebige Stiftleiste, Raster: 2.54mm" (at 203.2 66.675 0)
+      (effects (font (size 1.27 1.27)) hide)
+    )
     (pin "1")
     (pin "2")
@@
       (effects (font (size 1.27 1.27)) hide)
     )
+    (property "Reichelt" "" (at 35.56 115.57 0)
+      (effects (font (size 1.27 1.27)) hide)
+    )
     (pin "1")
     (pin "2")
@@
     )
     (property "Datasheet" "" (at 67.31 41.91 0)
+      (effects (font (size 1.27 1.27)) hide)
+    )
+    (property "Reichelt" "" (at 67.31 41.91 0)
+      (effects (font (size 1.27 1.27)) hide)
+    )
+    (property "Mouser" "RN73H1JTTD5101F100" (at 67.31 41.91 0)
+      (effects (font (size 1.27 1.27)) hide)
+    )
+    (property "Mouser Price/Stock" "https://www.mouser.at/ProductDetail/KOA-Speer/RN73H1JTTD5101F100?qs=Tw8F%252BABiY2owhjU7td4KeQ%3D%3D" (at 67.31 41.91 0)
       (effects (font (size 1.27 1.27)) hide)
     )
@@
       (effects (font (size 1.27 1.27)) hide)
     )
+    (property "Mouser" "13019315" (at 238.76 114.3 0)
+      (effects (font (size 1.27 1.27)) hide)
+    )
+    (property "Mouser Price/Stock" "https://www.mouser.at/ProductDetail/Schurter/1301.9315?qs=tGaZrb6HVSaeSttQbZxh%2FA%3D%3D" (at 238.76 114.3 0)
+      (effects (font (size 1.27 1.27)) hide)
+    )
+    (property "Reichelt" "" (at 238.76 114.3 0)
+      (effects (font (size 1.27 1.27)) hide)
+    )
     (pin "1")
     (pin "2")
@@
       (effects (font (size 1.27 1.27)) hide)
     )
+    (property "Mouser" "13019315" (at 195.58 110.49 0)
+      (effects (font (size 1.27 1.27)) hide)
+    )
+    (property "Mouser Price/Stock" "https://www.mouser.at/ProductDetail/Schurter/1301.9315?qs=tGaZrb6HVSaeSttQbZxh%2FA%3D%3D" (at 195.58 110.49 0)
+      (effects (font (size 1.27 1.27)) hide)
+    )
+    (property "Reichelt" "" (at 195.58 110.49 0)
+      (effects (font (size 1.27 1.27)) hide)
+    )

Commit message: Updated BOM
Parts:
- C5: Digikey 1276-CL10B104KB8NNNLCT-ND -> 1276-CL10B104KB8NNNLCT
- C5: Mouser (none) -> 81-GRM188R60J226ME0J
- C5: Mouser C0603C150F8HACAUTO -> 80-C0603C150F8HAUTO
- C5: Mouser F921E105KPA -> 647-F921E105KPA
- D2: Mouser 824015 -> 710-824015
- FL1: Mouser 744232090 -> 710-744232090
- J2: Mouser USB4105-GF-A -> 640-USB4105-GF-A
- R10: Mouser RN73H1JTTD5101F100 -> 791-RMC1/16K5101FTP
- R11: value 10k -> 10k/1%; Mouser (none) -> 660-RN73H1JT1002F100
- S1, S2: Mouser 13019315 -> 179-TS046643BK160SMT
- U3: Mouser ESP32-S3-WROOM-1-N8 -> 356-ESP32-S3WRM1N8R2
- Y1: Mouser ASDK-32.768KHz-LRT -> 815-ASDK-32.7K-LRT
Changed lines of the file:
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@@
       (effects (font (size 1.27 1.27)) hide)
     )
-    (property "Digikey" "1276-CL10B104KB8NNNLCT-ND" (at 121.92 95.25 0)
+    (property "Digikey" "1276-CL10B104KB8NNNLCT" (at 121.92 95.25 0)
       (effects (font (size 1.27 1.27)) hide)
     )
@@
       (effects (font (size 1.27 1.27)) hide)
     )
-    (property "Digikey" "1276-CL10B104KB8NNNLCT-ND" (at 238.76 119.38 0)
+    (property "Digikey" "1276-CL10B104KB8NNNLCT" (at 238.76 119.38 0)
       (effects (font (size 1.27 1.27)) hide)
     )
@@
       (effects (font (size 1.27 1.27)) hide)
     )
-    (property "Datasheet" "https://www.usb.org/sites/default/files/documents/usb_type-c.zip" (at 46.99 49.53 0)
-      (effects (font (size 1.27 1.27)) hide)
-    )
-    (property "Mouser" "USB4105-GF-A" (at 43.18 49.53 0)
+    (property "Datasheet" "https://www.mouser.at/ProductDetail/GCT/USB4105-GF-A?qs=KUoIvG%2F9IlY%2FMLlBMpStpA%3D%3D&gad_source=1&gclid=Cj0KCQiAyKurBhD5ARIsALamXaHB1WqEL8FpCW_cEPz8SMNbaXEcthQ5WIWoRdPENYKDcg-3_OVy5qsaArQwEALw_wcB" (at 46.99 49.53 0)
+      (effects (font (size 1.27 1.27)) hide)
+    )
+    (property "Mouser" "640-USB4105-GF-A" (at 43.18 49.53 0)
       (effects (font (size 1.27 1.27)) hide)
     )
@@
       (effects (font (size 1.27 1.27)) hide)
     )
-    (property "Mouser" "RN73H1JTTD5101F100" (at 67.31 39.37 0)
+    (property "Mouser" "791-RMC1/16K5101FTP" (at 67.31 39.37 0)
       (effects (font (size 1.27 1.27)) hide)
     )
@@
       (effects (font (size 1.27 1.27)) hide)
     )
-    (property "Mouser" "824015" (at 110.49 50.8 0)
+    (property "Mouser" "710-824015" (at 110.49 50.8 0)
       (effects (font (size 1.27 1.27)) hide)
     )
@@
       (effects (font (size 1.27 1.27)) hide)
     )
+    (property "Mouser" "81-GRM188R60J226ME0J" (at 114.3 95.25 0)
+      (effects (font (size 1.27 1.27)) hide)
+    )
     (pin "1")
     (pin "2")
@@
       (effects (font (size 1.27 1.27)) hide)
     )
-    (property "Mouser" "ESP32-S3-WROOM-1-N8" (at 105.41 144.78 0)
+    (property "Mouser" "356-ESP32-S3WRM1N8R2" (at 105.41 144.78 0)
       (effects (font (size 1.27 1.27)) hide)
     )
@@
       (effects (font (size 1.778 1.778)) (justify bottom))
     )
-    (property "Value" "10k" (at 251.714 106.68 0)
+    (property "Value" "10k/1%" (at 251.714 106.68 0)
       (effects (font (size 1.778 1.778)) (justify top))
     )
@@
     )
     (property "Reichelt" "" (at 250.19 106.68 0)
+      (effects (font (size 1.27 1.27)) hide)
+    )
+    (property "Mouser" "660-RN73H1JT1002F100" (at 250.19 106.68 0)
       (effects (font (size 1.27 1.27)) hide)
     )
@@
       (effects (font (size 1.27 1.27)) hide)
     )
-    (property "Mouser" "744232090" (at 151.13 50.8 0)
+    (property "Mouser" "710-744232090" (at 151.13 50.8 0)
       (effects (font (size 1.27 1.27)) hide)
     )
@@
       (effects (font (size 1.27 1.27)) hide)
     )
-    (property "Mouser" "C0603C150F8HACAUTO" (at 35.56 120.65 90)
+    (property "Mouser" "80-C0603C150F8HAUTO" (at 35.56 120.65 90)
       (effects (font (size 1.27 1.27)) hide)
     )
@@
       (effects (font (size 1.27 1.27)) hide)
     )
-    (property "Mouser" "F921E105KPA" (at 250.19 118.11 0)
+    (property "Mouser" "647-F921E105KPA" (at 250.19 118.11 0)
       (effects (font (size 1.27 1.27)) hide)
     )
@@
       (effects (font (size 1.27 1.27)) hide)
     )
-    (property "Mouser" "ASDK-32.768KHz-LRT" (at 40.64 118.11 0)
+    (property "Mouser" "815-ASDK-32.7K-LRT" (at 40.64 118.11 0)
       (effects (font (size 1.27 1.27)) hide)
     )
@@
       (effects (font (size 1.27 1.27)) hide)
     )
-    (property "Mouser" "C0603C150F8HACAUTO" (at 35.56 115.57 90)
+    (property "Mouser" "80-C0603C150F8HAUTO" (at 35.56 115.57 90)
       (effects (font (size 1.27 1.27)) hide)
     )
@@
       (effects (font (size 1.27 1.27)) hide)
     )
-    (property "Mouser" "RN73H1JTTD5101F100" (at 67.31 41.91 0)
+    (property "Mouser" "791-RMC1/16K5101FTP" (at 67.31 41.91 0)
       (effects (font (size 1.27 1.27)) hide)
     )
@@
       (effects (font (size 1.27 1.27)) hide)
     )
-    (property "Mouser" "13019315" (at 238.76 114.3 0)
+    (property "Mouser" "179-TS046643BK160SMT" (at 238.76 114.3 0)
       (effects (font (size 1.27 1.27)) hide)
     )
@@
       (effects (font (size 1.27 1.27)) hide)
     )
-    (property "Mouser" "13019315" (at 195.58 110.49 0)
-      (effects (font (size 1.27 1.27)) hide)
-    )
+    (property "Mouser" "179-TS046643BK160SMT" (at 195.58 110.49 0)
+      (effects (font (size 1.27 1.27)) hide)
+    )

Commit message: Updated BOM
Parts:
- C5: Digikey 1276-CL10B104KB8NNNLCT -> 1276-CL10B104KB8NNNLCT-ND
- C5: Mouser 81-GRM188R60J226ME0J -> (none)
- C5: Mouser 80-C0603C150F8HAUTO -> C0603C150F8HACAUTO
- C5: Mouser 647-F921E105KPA -> F921E105KPA
- D2: Mouser 710-824015 -> 824015
- FL1: Mouser 710-744232090 -> 744232090
- J2: Mouser 640-USB4105-GF-A -> USB4105-GF-A
- R10: Mouser 791-RMC1/16K5101FTP -> RN73H1JTTD5101F100
- R11: value 10k/1% -> 10k; Mouser 660-RN73H1JT1002F100 -> (none)
- S1, S2: Mouser 179-TS046643BK160SMT -> 13019315
- U3: Mouser 356-ESP32-S3WRM1N8R2 -> ESP32-S3-WROOM-1-N8
- Y1: Mouser 815-ASDK-32.7K-LRT -> ABS07
Changed lines of the file:
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@@
       (effects (font (size 1.27 1.27)) hide)
     )
-    (property "Digikey" "1276-CL10B104KB8NNNLCT" (at 121.92 95.25 0)
+    (property "Digikey" "1276-CL10B104KB8NNNLCT-ND" (at 121.92 95.25 0)
       (effects (font (size 1.27 1.27)) hide)
     )
@@
       (effects (font (size 1.27 1.27)) hide)
     )
-    (property "Digikey" "1276-CL10B104KB8NNNLCT" (at 238.76 119.38 0)
+    (property "Digikey" "1276-CL10B104KB8NNNLCT-ND" (at 238.76 119.38 0)
       (effects (font (size 1.27 1.27)) hide)
     )
@@
       (effects (font (size 1.27 1.27)) hide)
     )
-    (property "Datasheet" "https://www.mouser.at/ProductDetail/GCT/USB4105-GF-A?qs=KUoIvG%2F9IlY%2FMLlBMpStpA%3D%3D&gad_source=1&gclid=Cj0KCQiAyKurBhD5ARIsALamXaHB1WqEL8FpCW_cEPz8SMNbaXEcthQ5WIWoRdPENYKDcg-3_OVy5qsaArQwEALw_wcB" (at 46.99 49.53 0)
-      (effects (font (size 1.27 1.27)) hide)
-    )
-    (property "Mouser" "640-USB4105-GF-A" (at 43.18 49.53 0)
+    (property "Datasheet" "https://www.usb.org/sites/default/files/documents/usb_type-c.zip" (at 46.99 49.53 0)
+      (effects (font (size 1.27 1.27)) hide)
+    )
+    (property "Mouser" "USB4105-GF-A" (at 43.18 49.53 0)
       (effects (font (size 1.27 1.27)) hide)
     )
@@
       (effects (font (size 1.27 1.27)) hide)
     )
-    (property "Mouser" "791-RMC1/16K5101FTP" (at 67.31 39.37 0)
+    (property "Mouser" "RN73H1JTTD5101F100" (at 67.31 39.37 0)
       (effects (font (size 1.27 1.27)) hide)
     )
@@
       (effects (font (size 1.27 1.27)) hide)
     )
-    (property "Mouser" "710-824015" (at 110.49 50.8 0)
+    (property "Mouser" "824015" (at 110.49 50.8 0)
       (effects (font (size 1.27 1.27)) hide)
     )
@@
       (effects (font (size 1.27 1.27)) hide)
     )
-    (property "Mouser" "81-GRM188R60J226ME0J" (at 114.3 95.25 0)
-      (effects (font (size 1.27 1.27)) hide)
-    )
     (pin "1")
     (pin "2")
@@
       (effects (font (size 1.27 1.27)) hide)
     )
-    (property "Mouser" "356-ESP32-S3WRM1N8R2" (at 105.41 144.78 0)
+    (property "Mouser" "ESP32-S3-WROOM-1-N8" (at 105.41 144.78 0)
       (effects (font (size 1.27 1.27)) hide)
     )
@@
       (effects (font (size 1.778 1.778)) (justify bottom))
     )
-    (property "Value" "10k/1%" (at 251.714 106.68 0)
+    (property "Value" "10k" (at 251.714 106.68 0)
       (effects (font (size 1.778 1.778)) (justify top))
     )
@@
     )
     (property "Reichelt" "" (at 250.19 106.68 0)
-      (effects (font (size 1.27 1.27)) hide)
-    )
-    (property "Mouser" "660-RN73H1JT1002F100" (at 250.19 106.68 0)
       (effects (font (size 1.27 1.27)) hide)
     )
@@
       (effects (font (size 1.27 1.27)) hide)
     )
-    (property "Mouser" "710-744232090" (at 151.13 50.8 0)
+    (property "Mouser" "744232090" (at 151.13 50.8 0)
       (effects (font (size 1.27 1.27)) hide)
     )
@@
       (effects (font (size 1.27 1.27)) hide)
     )
-    (property "Mouser" "80-C0603C150F8HAUTO" (at 35.56 120.65 90)
+    (property "Mouser" "C0603C150F8HACAUTO" (at 35.56 120.65 90)
       (effects (font (size 1.27 1.27)) hide)
     )
@@
       (effects (font (size 1.27 1.27)) hide)
     )
-    (property "Mouser" "647-F921E105KPA" (at 250.19 118.11 0)
+    (property "Mouser" "F921E105KPA" (at 250.19 118.11 0)
       (effects (font (size 1.27 1.27)) hide)
     )
@@
       (effects (font (size 1.27 1.27)) hide)
     )
-    (property "Mouser" "815-ASDK-32.7K-LRT" (at 40.64 118.11 0)
+    (property "Mouser" "ABS07" (at 40.64 118.11 0)
       (effects (font (size 1.27 1.27)) hide)
     )
@@
       (effects (font (size 1.27 1.27)) hide)
     )
-    (property "Mouser" "80-C0603C150F8HAUTO" (at 35.56 115.57 90)
+    (property "Mouser" "C0603C150F8HACAUTO" (at 35.56 115.57 90)
       (effects (font (size 1.27 1.27)) hide)
     )
@@
       (effects (font (size 1.27 1.27)) hide)
     )
-    (property "Mouser" "791-RMC1/16K5101FTP" (at 67.31 41.91 0)
+    (property "Mouser" "RN73H1JTTD5101F100" (at 67.31 41.91 0)
       (effects (font (size 1.27 1.27)) hide)
     )
@@
       (effects (font (size 1.27 1.27)) hide)
     )
-    (property "Mouser" "179-TS046643BK160SMT" (at 238.76 114.3 0)
+    (property "Mouser" "13019315" (at 238.76 114.3 0)
       (effects (font (size 1.27 1.27)) hide)
     )
@@
       (effects (font (size 1.27 1.27)) hide)
     )
-    (property "Mouser" "179-TS046643BK160SMT" (at 195.58 110.49 0)
-      (effects (font (size 1.27 1.27)) hide)
-    )
+    (property "Mouser" "13019315" (at 195.58 110.49 0)
+      (effects (font (size 1.27 1.27)) hide)
+    )
