File: Hardware/HM_mainboard/Microcontroller.kicad_sch (KiCad schematic)
At the start: 19 parts, among them J2 USB4105-GF-A, J3 Conn_01x04, U3 ESP32-S3-WROOM-1, Y1 32.768 kHz

Commit message: Added BOM, PDF and zipped V2.0.0 project data
Parts:
- removed J3: Conn_01x04, Connector_PinHeader_2.54mm:PinHeader_1x04_P2.54mm_Vertical, symbol Connector_Generic:Conn_01x04
Other:
- note added: "Manual-Reset (internal)"
- note removed: "Manual-Reset"
- note removed: "UART Pin-Header"
Changed lines of the file:
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@@
-    (stroke (width 0) (type default))
-  )
-  (wire (pts (xy 197.485 62.23) (xy 197.485 64.135))
     (stroke (width 0) (type default))
   )
@@
     (stroke (width 0) (type default))
   )
-  (wire (pts (xy 193.04 69.215) (xy 200.025 69.215))
-    (stroke (width 0) (type default))
-  )
   (wire (pts (xy 43.18 72.39) (xy 43.18 73.66))
     (stroke (width 0) (type default))
@@
     (stroke (width 0) (type default))
   )
-  (wire (pts (xy 193.04 66.675) (xy 200.025 66.675))
-    (stroke (width 0) (type default))
-  )
   (wire (pts (xy 195.58 139.065) (xy 195.58 141.605))
     (stroke (width 0.1524) (type solid))
@@
     (stroke (width 0) (type default))
   )
-  (wire (pts (xy 197.485 64.135) (xy 200.025 64.135))
-    (stroke (width 0) (type default))
-  )
   (wire (pts (xy 146.05 53.34) (xy 132.08 53.34))
     (stroke (width 0) (type default))
@@
     (stroke (width 0) (type default))
   )
-  (wire (pts (xy 197.485 71.755) (xy 200.025 71.755))
-    (stroke (width 0) (type default))
-  )
-  (wire (pts (xy 197.485 74.295) (xy 197.485 71.755))
-    (stroke (width 0) (type default))
-  )
   (wire (pts (xy 151.13 172.72) (xy 153.67 172.72))
     (stroke (width 0) (type default))
@@
   )
   (rectangle (start 177.165 83.82) (end 261.62 110.49)
-    (stroke (width 0) (type default))
-    (fill (type none))
-  )
-  (rectangle (start 177.165 48.26) (end 222.885 81.28)
     (stroke (width 0) (type default))
     (fill (type none))
@@
     (effects (font (size 1.27 1.27)) (justify left top))
   )
-  (text "UART Pin-Header" (at 179.705 54.61 0)
-    (effects (font (size 2.54 2.159) (thickness 0.4318) bold) (justify left bottom))
-  )
   (text "USB-C Plug for flashing and battery charging\n" (at 20.32 21.59 0)
     (effects (font (size 2.54 2.159) (thickness 0.4318) bold) (justify left bottom))
@@
     (effects (font (size 2.54 2.159)) (justify left bottom))
   )
-  (text "Manual-Reset" (at 179.705 120.015 0)
+  (text "Manual-Reset (internal)\n" (at 179.705 120.015 0)
     (effects (font (size 2.54 2.159) (thickness 0.4318) bold) (justify left bottom))
   )
@@
     (effects (font (size 1.27 1.27)) (justify left bottom))
   )
-  (label "UART_RXD" (at 193.04 69.215 180) (fields_autoplaced)
-    (effects (font (size 1.27 1.27)) (justify right bottom))
-  )
   (label "USB_C_D+" (at 153.67 116.84 0) (fields_autoplaced)
     (effects (font (size 1.27 1.27)) (justify left bottom))
@@
   (label "BOOT" (at 154.94 124.46 0) (fields_autoplaced)
     (effects (font (size 1.27 1.27)) (justify left bottom))
-  )
-  (label "UART_TXD" (at 193.04 66.675 180) (fields_autoplaced)
-    (effects (font (size 1.27 1.27)) (justify right bottom))
   )
   (label "USB_C_D+" (at 162.56 53.34 0) (fields_autoplaced)
@@
         (path "/64c5aff3-bdec-4fb6-b5ec-87e5efa2adf7"
           (reference "#SUPPLY14") (unit 1)
-        )
-      )
-    )
-  )
-  (symbol (lib_name "GND_1") (lib_id "power:GND") (at 197.485 74.295 0) (unit 1)
-    (in_bom yes) (on_board yes) (dnp no)
-    (property "Reference" "#PWR06" (at 197.485 80.645 0)
-      (effects (font (size 1.27 1.27)) hide)
-    )
-    (property "Value" "GND" (at 197.485 78.105 0)
-      (effects (font (size 1.27 1.27)))
-    )
-    (property "Footprint" "" (at 197.485 74.295 0)
-      (effects (font (size 1.27 1.27)) hide)
-    )
-    (property "Datasheet" "" (at 197.485 74.295 0)
-      (effects (font (size 1.27 1.27)) hide)
-    )
-    (pin "1")
-    (instances
-      (project "HM_mainboard"
-        (path "/54a6df43-5475-46a2-9916-8b0260700d4c"
-          (reference "#PWR06") (unit 1)
-        )
-        (path "/54a6df43-5475-46a2-9916-8b0260700d4c/8a725ce3-408a-4762-9df2-b56094186e56"
-          (reference "#PWR016") (unit 1)
-        )
-        (path "/54a6df43-5475-46a2-9916-8b0260700d4c/9043a365-e24a-41b8-9f6d-decb4da0da6a"
-          (reference "#PWR010") (unit 1)
-        )
-        (path "/54a6df43-5475-46a2-9916-8b0260700d4c/137c5701-d01e-40ce-919d-b371cfda41da"
-          (reference "#PWR01") (unit 1)
         )
       )
@@
     )
   )
-  (symbol (lib_id "esp32-thing-eagle-import:3.3V") (at 197.485 62.23 0) (unit 1)
-    (in_bom yes) (on_board yes) (dnp no)
-    (property "Reference" "#SUPPLY08" (at 197.485 62.23 0)
-      (effects (font (size 1.27 1.27)) hide)
-    )
-    (property "Value" "3.3V" (at 196.469 58.674 0)
-      (effects (font (size 1.778 1.5113)) (justify left bottom))
-    )
-    (property "Footprint" "" (at 197.485 62.23 0)
-      (effects (font (size 1.27 1.27)) hide)
-    )
-    (property "Datasheet" "" (at 197.485 62.23 0)
-      (effects (font (size 1.27 1.27)) hide)
-    )
-    (pin "1")
-    (instances
-      (project "HM_mainboard"
-        (path "/54a6df43-5475-46a2-9916-8b0260700d4c"
-          (reference "#SUPPLY08") (unit 1)
-        )
-        (path "/54a6df43-5475-46a2-9916-8b0260700d4c/8a725ce3-408a-4762-9df2-b56094186e56"
-          (reference "#SUPPLY012") (unit 1)
-        )
-      )
-      (project "esp32-thing"
-        (path "/64c5aff3-bdec-4fb6-b5ec-87e5efa2adf7"
-          (reference "#SUPPLY8") (unit 1)
-        )
-      )
-    )
-  )
   (symbol (lib_id "Device:C") (at 35.56 120.65 90) (unit 1)
     (in_bom yes) (on_board yes) (dnp no)
@@
         )
       )
-    )
-  )
-  (symbol (lib_id "Connector_Generic:Conn_01x04") (at 205.105 66.675 0) (unit 1)
-    (in_bom yes) (on_board yes) (dnp no) (fields_autoplaced)
-    (property "Reference" "J3" (at 208.28 66.675 0)
-      (effects (font (size 1.27 1.27)) (justify left))
-    )
-    (property "Value" "Conn_01x04" (at 208.28 69.215 0)
-      (effects (font (size 1.27 1.27)) (justify left))
-    )
-    (property "Footprint" "Connector_PinHeader_2.54mm:PinHeader_1x04_P2.54mm_Vertical" (at 205.105 66.675 0)
-      (effects (font (size 1.27 1.27)) hide)
-    )
-    (property "Datasheet" "~" (at 205.105 66.675 0)
-      (effects (font (size 1.27 1.27)) hide)
-    )
-    (property "Reichelt" "" (at 205.105 66.675 0)
-      (effects (font (size 1.27 1.27)) hide)
-    )
-    (property "Mouser" "Beliebige Stiftleiste, Raster: 2.54mm" (at 205.105 66.675 0)
-      (effects (font (size 1.27 1.27)) hide)
-    )
-    (pin "1")
-    (pin "2")
-    (pin "3")
-    (pin "4")
-    (instances
-      (project "HM_mainboard"
-        (path "/54a6df43-5475-46a2-9916-8b0260700d4c/8a725ce3-408a-4762-9df2-b56094186e56"
-          (reference "J3") (unit 1)
-        )
-      )
