File: Hardware/HM_mainboard/untitled.kicad_sch (KiCad schematic)
At the start: 17 parts, among them J1 JST PH2P ST90, Q1 PMOS AS3401, U1 MCP73831-2, U2 TC1262-33

Commit message: updated schematic
Parts:
- added D3: 155124RV73200, HeadMouse:155124RV73200, symbol Device:LED_Dual_KAK
Connections:
- net BATT_CHARGING_STATUS: now also D3.1 (K1), D3.3 (K2); no longer R6.1
- new net: D3.2 (A), R6.1
Other:
- moved on the sheet: R6
Changed lines of the file:
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@@
   (junction (at 109.855 149.86) (diameter 0) (color 0 0 0 0)
   )
+  (junction (at 128.905 149.86) (diameter 0) (color 0 0 0 0)
+  )
   (junction (at 59.69 65.405) (diameter 0) (color 0 0 0 0)
   )
@@
   (junction (at 200.66 138.43) (diameter 0) (color 0 0 0 0)
   )
-  (junction (at 128.27 149.86) (diameter 0) (color 0 0 0 0)
-  )
   (junction (at 65.405 146.05) (diameter 0) (color 0 0 0 0)
   )
@@
   (junction (at 49.53 57.785) (diameter 0) (color 0 0 0 0)
   )
+  (junction (at 133.985 149.86) (diameter 0) (color 0 0 0 0)
+  )
   (wire (pts (xy 63.5 155.575) (xy 65.405 155.575))
     (stroke (width 0) (type default))
@@
     (stroke (width 0.1524) (type solid))
   )
-  (wire (pts (xy 128.27 147.32) (xy 128.27 149.86))
-    (stroke (width 0) (type default))
-  )
   (wire (pts (xy 200.66 123.19) (xy 200.66 125.73))
     (stroke (width 0) (type default))
@@
     (stroke (width 0.1524) (type solid))
   )
-  (wire (pts (xy 109.855 149.86) (xy 128.27 149.86))
-    (stroke (width 0) (type default))
-  )
   (wire (pts (xy 97.79 120.65) (xy 97.79 139.7))
     (stroke (width 0) (type default))
@@
     (stroke (width 0) (type default))
   )
-  (wire (pts (xy 114.935 119.38) (xy 114.935 120.65))
+  (wire (pts (xy 114.935 118.11) (xy 114.935 120.65))
     (stroke (width 0) (type default))
   )
@@
     (stroke (width 0.1524) (type solid))
   )
+  (wire (pts (xy 133.985 147.955) (xy 133.985 149.86))
+    (stroke (width 0) (type default))
+  )
   (wire (pts (xy 57.15 65.405) (xy 59.69 65.405))
     (stroke (width 0) (type default))
@@
     (stroke (width 0) (type default))
   )
-  (wire (pts (xy 128.27 134.62) (xy 128.27 137.16))
+  (wire (pts (xy 128.905 149.86) (xy 133.985 149.86))
+    (stroke (width 0) (type default))
+  )
+  (wire (pts (xy 131.445 130.175) (xy 131.445 132.715))
+    (stroke (width 0) (type default))
+  )
+  (wire (pts (xy 131.445 118.11) (xy 131.445 120.015))
     (stroke (width 0) (type default))
   )
@@
     (stroke (width 0) (type default))
   )
+  (wire (pts (xy 128.905 147.955) (xy 128.905 149.86))
+    (stroke (width 0) (type default))
+  )
   (wire (pts (xy 200.66 153.67) (xy 200.66 151.13))
     (stroke (width 0) (type default))
@@
     (stroke (width 0.1524) (type solid))
   )
-  (wire (pts (xy 132.08 149.86) (xy 128.27 149.86))
+  (wire (pts (xy 109.855 149.86) (xy 128.905 149.86))
+    (stroke (width 0) (type default))
+  )
+  (wire (pts (xy 133.985 149.86) (xy 139.065 149.86))
     (stroke (width 0) (type default))
   )
@@
     (effects (font (size 2.54 2.54) (thickness 0.508) bold) (justify left bottom))
   )
-  (hierarchical_label "BATT_CHARGING_STATUS" (shape input) (at 132.08 149.86 0) (fields_autoplaced)
+  (hierarchical_label "BATT_CHARGING_STATUS" (shape input) (at 139.065 149.86 0) (fields_autoplaced)
     (effects (font (size 1.27 1.27)) (justify left))
   )
@@
     )
   )
-  (symbol (lib_id "esp32-thing-eagle-import:V_USB") (at 114.935 119.38 0) (mirror y) (unit 1)
-    (in_bom yes) (on_board yes) (dnp no)
-    (property "Reference" "#SUPPLY06" (at 114.935 119.38 0)
-      (effects (font (size 1.27 1.27)) hide)
-    )
-    (property "Value" "V_USB" (at 115.951 115.824 0)
+  (symbol (lib_id "esp32-thing-eagle-import:V_USB") (at 114.935 118.11 0) (mirror y) (unit 1)
+    (in_bom yes) (on_board yes) (dnp no)
+    (property "Reference" "#SUPPLY06" (at 114.935 118.11 0)
+      (effects (font (size 1.27 1.27)) hide)
+    )
+    (property "Value" "V_USB" (at 115.951 114.554 0)
       (effects (font (size 1.778 1.5113)) (justify left bottom))
     )
-    (property "Footprint" "" (at 114.935 119.38 0)
-      (effects (font (size 1.27 1.27)) hide)
-    )
-    (property "Datasheet" "" (at 114.935 119.38 0)
+    (property "Footprint" "" (at 114.935 118.11 0)
+      (effects (font (size 1.27 1.27)) hide)
+    )
+    (property "Datasheet" "" (at 114.935 118.11 0)
       (effects (font (size 1.27 1.27)) hide)
     )
@@
     )
   )
+  (symbol (lib_id "Device:LED_Dual_KAK") (at 131.445 140.335 270) (unit 1)
+    (in_bom yes) (on_board yes) (dnp no) (fields_autoplaced)
+    (property "Reference" "D3" (at 139.065 139.1285 90)
+      (effects (font (size 1.27 1.27)) (justify left))
+    )
+    (property "Value" "155124RV73200" (at 139.065 141.6685 90)
+      (effects (font (size 1.27 1.27)) (justify left))
+    )
+    (property "Footprint" "HeadMouse:155124RV73200" (at 131.445 141.605 0)
+      (effects (font (size 1.27 1.27)) hide)
+    )
+    (property "Datasheet" "https://www.we-online.com/components/products/datasheet/155124RV73200.pdf" (at 131.445 141.605 0)
+      (effects (font (size 1.27 1.27)) hide)
+    )
+    (property "Mouser" "155124RV73200" (at 131.445 140.335 0)
+      (effects (font (size 1.27 1.27)) hide)
+    )
+    (property "Mouser Price/Stock" "https://www.mouser.at/ProductDetail/Wurth-Elektronik/155124RV73200?qs=5aG0NVq1C4yQQzqaqWGYAg%3D%3D" (at 131.445 140.335 0)
+      (effects (font (size 1.27 1.27)) hide)
+    )
+    (property "Reichelt" "" (at 131.445 140.335 0)
+      (effects (font (size 1.27 1.27)) hide)
+    )
+    (pin "1")
+    (pin "2")
+    (pin "3")
+    (instances
+      (project "HM_mainboard"
+        (path "/54a6df43-5475-46a2-9916-8b0260700d4c/137c5701-d01e-40ce-919d-b371cfda41da"
+          (reference "D3") (unit 1)
+        )
+        (path "/54a6df43-5475-46a2-9916-8b0260700d4c/b19d5209-4861-4a96-a3d1-daca4a23de52"
+          (reference "D5") (unit 1)
+        )
+      )
+    )
+  )
   (symbol (lib_name "GND_1") (lib_id "power:GND") (at 63.5 157.48 0) (unit 1)
     (in_bom yes) (on_board yes) (dnp no) (fields_autoplaced)
@@
     )
   )
-  (symbol (lib_id "esp32-thing-eagle-import:27OHM1/10W1%(0603)0603-RES") (at 128.27 142.24 90) (unit 1)
-    (in_bom yes) (on_board yes) (dnp no)
-    (property "Reference" "R6" (at 126.7714 146.812 0)
+  (symbol (lib_id "esp32-thing-eagle-import:27OHM1/10W1%(0603)0603-RES") (at 131.445 125.095 90) (unit 1)
+    (in_bom yes) (on_board yes) (dnp no)
+    (property "Reference" "R6" (at 129.9464 129.667 0)
       (effects (font (size 1.778 1.778)) (justify left bottom))
     )
-    (property "Value" "1k" (at 127 140.97 0)
+    (property "Value" "1k" (at 130.175 123.825 0)
       (effects (font (size 1.778 1.778)) (justify left bottom))
     )
-    (property "Footprint" "Resistor_SMD:R_0603_1608Metric_Pad0.98x0.95mm_HandSolder" (at 128.27 142.24 0)
-      (effects (font (size 1.27 1.27)) hide)
-    )
-    (property "Datasheet" "" (at 128.27 142.24 0)
-      (effects (font (size 1.27 1.27)) hide)
-    )
-    (property "Mouser" "ERJ-PA3J121V" (at 128.27 142.24 0)
-      (effects (font (size 1.27 1.27)) hide)
-    )
-    (property "Reichelt" "" (at 128.27 142.24 0)
+    (property "Footprint" "Resistor_SMD:R_0603_1608Metric_Pad0.98x0.95mm_HandSolder" (at 131.445 125.095 0)
+      (effects (font (size 1.27 1.27)) hide)
+    )
+    (property "Datasheet" "" (at 131.445 125.095 0)
+      (effects (font (size 1.27 1.27)) hide)
+    )
+    (property "Mouser" "ERJ-PA3J121V" (at 131.445 125.095 0)
+      (effects (font (size 1.27 1.27)) hide)
+    )
+    (property "Reichelt" "" (at 131.445 125.095 0)
       (effects (font (size 1.27 1.27)) hide)
     )
@@
     )
   )
-  (symbol (lib_id "esp32-thing-eagle-import:V_BATT") (at 128.27 134.62 0) (unit 1)
-    (in_bom yes) (on_board yes) (dnp no)
-    (property "Reference" "#SUPPLY02" (at 128.27 134.62 0)
-      (effects (font (size 1.27 1.27)) hide)
-    )
-    (property "Value" "V_BATT" (at 127.254 131.064 0)
+  (symbol (lib_id "esp32-thing-eagle-import:V_BATT") (at 131.445 118.11 0) (unit 1)
+    (in_bom yes) (on_board yes) (dnp no)
+    (property "Reference" "#SUPPLY02" (at 131.445 118.11 0)
+      (effects (font (size 1.27 1.27)) hide)
+    )
+    (property "Value" "V_BATT" (at 130.429 114.554 0)
       (effects (font (size 1.778 1.5113)) (justify left bottom))
     )
-    (property "Footprint" "" (at 128.27 134.62 0)
-      (effects (font (size 1.27 1.27)) hide)
-    )
-    (property "Datasheet" "" (at 128.27 134.62 0)
-      (effects (font (size 1.27 1.27)) hide)
-    )
+    (property "Footprint" "" (at 131.445 118.11 0)
+      (effects (font (size 1.27 1.27)) hide)
+    )
+    (property "Datasheet" "" (at 131.445 118.11 0)
+      (effects (font (size 1.27 1.27)) hide)
+    )
